Commit message: Remove obsolete files and scripts related to the robot automation system, including documentation and demo scripts. Update CMakeLists.txt to reflect changes in package structure and improve build process. Adjust docker-compose.yml to ensure proper service configuration for the new setup.

File: ros2_ws/src/my_robot_description/urdf/my_robot.urdf.xacro (robot description, xacro)
@@ -122,6 +122,6 @@
   <xacro:omni_wheel name="wheel_2" x="${wheel_2_x}" y="${wheel_2_y}"/>
   <xacro:omni_wheel name="wheel_3" x="${wheel_3_x}" y="${wheel_3_y}"/>
-  <!-- Laser frame (RPLidar position) -->
-  <link name="laser_frame">
+  <!-- LIDAR frame -->
+  <link name="lidar_frame">
     <visual>
       <geometry>
@@ -146,9 +146,109 @@
     </inertial>
   </link>
-  <joint name="laser_joint" type="fixed">
+  <joint name="lidar_joint" type="fixed">
     <parent link="base_link"/>
-    <child link="laser_frame"/>
+    <child link="lidar_frame"/>
     <origin xyz="0 0 ${base_height + 0.05}" rpy="0 0 0"/>
   </joint>
+  <!-- Ultrasonic Sensors (4x) -->
+  <xacro:macro name="ultrasonic_sensor" params="name x y z">
+    <link name="${name}_link">
+      <visual>
+        <geometry>
+          <cylinder length="0.02" radius="0.015"/>
+        </geometry>
+        <material name="yellow">
+          <color rgba="1.0 1.0 0.0 1.0"/>
+        </material>
+        <origin xyz="0 0 0" rpy="0 0 0"/>
+      </visual>
+      <collision>
+        <geometry>
+          <cylinder length="0.02" radius="0.015"/>
+        </geometry>
+        <origin xyz="0 0 0" rpy="0 0 0"/>
+      </collision>
+      <inertial>
+        <mass value="0.05"/>
+        <inertia ixx="0.0001" ixy="0.0" ixz="0.0"
+                 iyy="0.0001" iyz="0.0"
+                 izz="0.0002"/>
+      </inertial>
+    </link>
+    <joint name="${name}_joint" type="fixed">
+      <parent link="base_link"/>
+      <child link="${name}_link"/>
+      <origin xyz="${x} ${y} ${z}" rpy="0 0 0"/>
+    </joint>
+  </xacro:macro>
+  <!-- IR Sharp Sensors (3x) -->
+  <xacro:macro name="ir_sensor" params="name x y z">
+    <link name="${name}_link">
+      <visual>
+        <geometry>
+          <box size="0.02 0.02 0.015"/>
+        </geometry>
+        <material name="orange">
+          <color rgba="1.0 0.5 0.0 1.0"/>
+        </material>
+        <origin xyz="0 0 0" rpy="0 0 0"/>
+      </visual>
+      <collision>
+        <geometry>
+          <box size="0.02 0.02 0.015"/>
+        </geometry>
+        <origin xyz="0 0 0" rpy="0 0 0"/>
+      </collision>
+      <inertial>
+        <mass value="0.03"/>
+        <inertia ixx="0.0001" ixy="0.0" ixz="0.0"
+                 iyy="0.0001" iyz="0.0"
+                 izz="0.0002"/>
+      </inertial>
+    </link>
+    <joint name="${name}_joint" type="fixed">
+      <parent link="base_link"/>
+      <child link="${name}_link"/>
+      <origin xyz="${x} ${y} ${z}" rpy="0 0 0"/>
+    </joint>
+  </xacro:macro>
+  <!-- Line Sensor -->
+  <link name="line_sensor_link">
+    <visual>
+      <geometry>
+        <box size="0.08 0.03 0.01"/>
+      </geometry>
+      <material name="purple">
+        <color rgba="0.8 0.0 0.8 1.0"/>
+      </material>
+      <origin xyz="0 0 0" rpy="0 0 0"/>
+    </visual>
+    <collision>
+      <geometry>
+        <box size="0.08 0.03 0.01"/>
+      </geometry>
+      <origin xyz="0 0 0" rpy="0 0 0"/>
+    </collision>
+    <inertial>
+      <mass value="0.02"/>
+      <inertia ixx="0.0001" ixy="0.0" ixz="0.0"
+               iyy="0.0001" iyz="0.0"
+               izz="0.0002"/>
+    </inertial>
+  </link>
+  <joint name="line_sensor_joint" type="fixed">
+    <parent link="base_link"/>
+    <child link="line_sensor_link"/>
+    <origin xyz="0 0 -${base_height/2 - 0.02}" rpy="0 0 0"/>
+  </joint>
+  <!-- Create ultrasonic sensors -->
+  <xacro:ultrasonic_sensor name="ultrasonic_front" x="${base_radius - 0.02}" y="0" z="${base_height/2}"/>
+  <xacro:ultrasonic_sensor name="ultrasonic_back" x="${-base_radius + 0.02}" y="0" z="${base_height/2}"/>
+  <xacro:ultrasonic_sensor name="ultrasonic_left" x="0" y="${base_radius - 0.02}" z="${base_height/2}"/>
+  <xacro:ultrasonic_sensor name="ultrasonic_right" x="0" y="${-base_radius + 0.02}" z="${base_height/2}"/>
+  <!-- Create IR sensors -->
+  <xacro:ir_sensor name="ir_front" x="${base_radius - 0.05}" y="0" z="${base_height/2}"/>
+  <xacro:ir_sensor name="ir_left" x="0" y="${base_radius - 0.05}" z="${base_height/2}"/>
+  <xacro:ir_sensor name="ir_right" x="0" y="${-base_radius + 0.05}" z="${base_height/2}"/>
   <!-- IMU frame -->
   <link name="imu_link">
@@ -205,4 +305,74 @@
     <origin xyz="${base_radius - 0.02} 0 ${base_height + 0.03}" rpy="0 0 0"/>
   </joint>
+  <!-- Lifter/Forklift (1x DC Motor + Encoder) -->
+  <link name="lifter_link">
+    <visual>
+      <geometry>
+        <box size="0.1 0.1 0.3"/>
+      </geometry>
+      <material name="silver">
+        <color rgba="0.7 0.7 0.7 1.0"/>
+      </material>
+      <origin xyz="0 0 0" rpy="0 0 0"/>
+    </visual>
+    <collision>
+      <geometry>
+        <box size="0.1 0.1 0.3"/>
+      </geometry>
+      <origin xyz="0 0 0" rpy="0 0 0"/>
+    </collision>
+    <inertial>
+      <mass value="2.0"/>
+      <inertia ixx="0.1" ixy="0.0" ixz="0.0"
+               iyy="0.1" iyz="0.0"
+               izz="0.05"/>
+    </inertial>
+  </link>
+  <joint name="lifter_joint" type="prismatic">
+    <parent link="base_link"/>
+    <child link="lifter_link"/>
+    <origin xyz="0 0 ${base_height/2}" rpy="0 0 0"/>
+    <axis xyz="0 0 1"/>
+    <limit effort="100.0" lower="0.0" upper="0.1" velocity="0.1"/>
+  </joint>
+  <!-- Servo Motors (5x) -->
+  <xacro:macro name="servo_joint" params="name x y z roll pitch yaw">
+    <link name="${name}_link">
+      <visual>
+        <geometry>
+          <box size="0.03 0.03 0.04"/>
+        </geometry>
+        <material name="blue">
+          <color rgba="0.0 0.3 0.8 1.0"/>
+        </material>
+        <origin xyz="0 0 0" rpy="0 0 0"/>
+      </visual>
+      <collision>
+        <geometry>
+          <box size="0.03 0.03 0.04"/>
+        </geometry>
+        <origin xyz="0 0 0" rpy="0 0 0"/>
+      </collision>
+      <inertial>
+        <mass value="0.1"/>
+        <inertia ixx="0.0001" ixy="0.0" ixz="0.0"
+                 iyy="0.0001" iyz="0.0"
+                 izz="0.0002"/>
+      </inertial>
+    </link>
+    <joint name="${name}_joint" type="revolute">
+      <parent link="lifter_link"/>
+      <child link="${name}_link"/>
+      <origin xyz="${x} ${y} ${z}" rpy="${roll} ${pitch} ${yaw}"/>
+      <axis xyz="0 0 1"/>
+      <limit effort="10.0" lower="-3.14159" upper="3.14159" velocity="1.0"/>
+    </joint>
+  </xacro:macro>
+  <!-- Create servo joints -->
+  <xacro:servo_joint name="servo_1" x="0.05" y="0" z="0.15" roll="0" pitch="0" yaw="0"/>
+  <xacro:servo_joint name="servo_2" x="0.08" y="0" z="0.15" roll="0" pitch="0" yaw="0"/>
+  <xacro:servo_joint name="servo_3" x="0.11" y="0" z="0.15" roll="0" pitch="0" yaw="0"/>
+  <xacro:servo_joint name="servo_4" x="0.14" y="0" z="0.15" roll="0" pitch="0" yaw="0"/>
+  <xacro:servo_joint name="servo_5" x="0.17" y="0" z="0.15" roll="0" pitch="0" yaw="0"/>
   <!-- Gazebo plugins -->
   <gazebo>
@@ -249,6 +419,6 @@
       <frame_name>imu_link</frame_name>
     </plugin>
-    <!-- Laser scan plugin -->
-    <plugin name="laser_plugin" filename="libgazebo_ros_ray_sensor.so">
+    <!-- LIDAR plugin -->
+    <plugin name="lidar_plugin" filename="libgazebo_ros_ray_sensor.so">
       <ros>
         <namespace></namespace>
@@ -256,7 +426,7 @@
       </ros>
       <always_on>true</always_on>
-      <update_rate>30.0</update_rate>
+      <update_rate>10.0</update_rate>
       <topic_name>scan</topic_name>
-      <frame_name>laser_frame</frame_name>
+      <frame_name>lidar_frame</frame_name>
       <ray>
         <scan>
@@ -270,6 +440,127 @@
         <range>
           <min>0.1</min>
-          <max>10.0</max>
+          <max>30.0</max>
           <resolution>0.01</resolution>
+        </range>
+      </ray>
+    </plugin>
+    <!-- Ultrasonic sensor plugins (4x) -->
+    <plugin name="ultrasonic_front_plugin" filename="libgazebo_ros_ray_sensor.so">
+      <ros>
+        <namespace></namespace>
+        <remapping>range:=/ultrasonic/front</remapping>
+      </ros>
+      <always_on>true</always_on>
+      <update_rate>10.0</update_rate>
+      <topic_name>range</topic_name>
+      <frame_name>ultrasonic_front_link</frame_name>
+      <ray>
+        <range>
+          <min>0.02</min>
+          <max>4.0</max>
+          <resolution>0.01</resolution>
+        </range>
+      </ray>
+    </plugin>
+    <plugin name="ultrasonic_back_plugin" filename="libgazebo_ros_ray_sensor.so">
+      <ros>
+        <namespace></namespace>
+        <remapping>range:=/ultrasonic/back</remapping>
+      </ros>
+      <always_on>true</always_on>
+      <update_rate>10.0</update_rate>
+      <topic_name>range</topic_name>
+      <frame_name>ultrasonic_back_link</frame_name>
+      <ray>
+        <range>
+          <min>0.02</min>
+          <max>4.0</max>
+          <resolution>0.01</resolution>
+        </range>
+      </ray>
+    </plugin>
+    <plugin name="ultrasonic_left_plugin" filename="libgazebo_ros_ray_sensor.so">
+      <ros>
+        <namespace></namespace>
+        <remapping>range:=/ultrasonic/left</remapping>
+      </ros>
+      <always_on>true</always_on>
+      <update_rate>10.0</update_rate>
+      <topic_name>range</topic_name>
+      <frame_name>ultrasonic_left_link</frame_name>
+      <ray>
+        <range>
+          <min>0.02</min>
+          <max>4.0</max>
+          <resolution>0.01</resolution>
+        </range>
+      </ray>
+    </plugin>
+    <plugin name="ultrasonic_right_plugin" filename="libgazebo_ros_ray_sensor.so">
+      <ros>
+        <namespace></namespace>
+        <remapping>range:=/ultrasonic/right</remapping>
+      </ros>
+      <always_on>true</always_on>
+      <update_rate>10.0</update_rate>
+      <topic_name>range</topic_name>
+      <frame_name>ultrasonic_right_link</frame_name>
+      <ray>
+        <range>
+          <min>0.02</min>
+          <max>4.0</max>
+          <resolution>0.01</resolution>
+        </range>
+      </ray>
+    </plugin>
+    <!-- IR Sharp sensor plugins (3x) -->
+    <plugin name="ir_front_plugin" filename="libgazebo_ros_ray_sensor.so">
+      <ros>
+        <namespace></namespace>
+        <remapping>range:=/ir/front</remapping>
+      </ros>
+      <always_on>true</always_on>
+      <update_rate>20.0</update_rate>
+      <topic_name>range</topic_name>
+      <frame_name>ir_front_link</frame_name>
+      <ray>
+        <range>
+          <min>0.04</min>
+          <max>0.8</max>
+          <resolution>0.001</resolution>
+        </range>
+      </ray>
+    </plugin>
+    <plugin name="ir_left_plugin" filename="libgazebo_ros_ray_sensor.so">
+      <ros>
+        <namespace></namespace>
+        <remapping>range:=/ir/left</remapping>
+      </ros>
+      <always_on>true</always_on>
+      <update_rate>20.0</update_rate>
+      <topic_name>range</topic_name>
+      <frame_name>ir_left_link</frame_name>
+      <ray>
+        <range>
+          <min>0.04</min>
+          <max>0.8</max>
+          <resolution>0.001</resolution>
+        </range>
+      </ray>
+    </plugin>
+    <plugin name="ir_right_plugin" filename="libgazebo_ros_ray_sensor.so">
+      <ros>
+        <namespace></namespace>
+        <remapping>range:=/ir/right</remapping>
+      </ros>
+      <always_on>true</always_on>
+      <update_rate>20.0</update_rate>
+      <topic_name>range</topic_name>
+      <frame_name>ir_right_link</frame_name>
+      <ray>
+        <range>
+          <min>0.04</min>
+          <max>0.8</max>
+          <resolution>0.001</resolution>
         </range>
       </ray>
