Commit message: Refactor robot automation scripts and workflows to enhance sensor integration and data handling. Updated JSON configurations for line and ultrasonic sensors, improved movement command logic for omni wheels, and added new API endpoints for IMU position and robot logs. Enhanced URDF model for hexagonal robot design, including updated sensor placements and properties, ensuring better performance and reliability in robot operations.

File: ros2_ws/src/my_robot_description/urdf/my_robot.urdf.xacro (robot description, xacro)
@@ -5,37 +5,47 @@
   <xacro:arg name="use_sim_time" default="true"/>
   <!-- Macros defined below -->
-  <!-- Robot base properties -->
+  <!-- Robot base properties - Hexagonal robot -->
   <xacro:property name="base_radius" value="0.3"/>
   <xacro:property name="base_height" value="0.15"/>
   <xacro:property name="wheel_radius" value="0.075"/>
   <xacro:property name="wheel_width" value="0.04"/>
-  <!-- Wheel positions for 3-wheeled omnidirectional robot -->
-  <!-- Wheels positioned at 120 degrees apart -->
-  <xacro:property name="wheel_1_x" value="${base_radius * 0.866}"/> <!-- cos(30°) -->
-  <xacro:property name="wheel_1_y" value="${base_radius * 0.5}"/>   <!-- sin(30°) -->
-  <xacro:property name="wheel_2_x" value="${-base_radius * 0.866}"/> <!-- -cos(30°) -->
-  <xacro:property name="wheel_2_y" value="${base_radius * 0.5}"/>   <!-- sin(30°) -->
-  <xacro:property name="wheel_3_x" value="0"/>
-  <xacro:property name="wheel_3_y" value="${-base_radius}"/>
-  <!-- Base link -->
+  <!-- Hexagonal shape properties -->
+  <xacro:property name="hexagon_side" value="0.25"/>
+  <!-- Wheel positions for 3-wheeled omnidirectional robot (lf, rf, b) -->
+  <!-- Front Left wheel -->
+  <xacro:property name="wheel_lf_x" value="${hexagon_side * 0.866}"/> <!-- cos(30°) -->
+  <xacro:property name="wheel_lf_y" value="${hexagon_side * 0.5}"/>   <!-- sin(30°) -->
+  <!-- Front Right wheel -->
+  <xacro:property name="wheel_rf_x" value="${-hexagon_side * 0.866}"/> <!-- -cos(30°) -->
+  <xacro:property name="wheel_rf_y" value="${hexagon_side * 0.5}"/>   <!-- sin(30°) -->
+  <!-- Back wheel -->
+  <xacro:property name="wheel_b_x" value="0"/>
+  <xacro:property name="wheel_b_y" value="${-hexagon_side}"/>
+  <!-- Base link - Hexagonal robot -->
   <link name="base_link">
     <visual>
       <geometry>
-        <cylinder length="${base_height}" radius="${base_radius}"/>
+        <!-- Hexagonal prism approximation using cylinder -->
+        <cylinder length="${base_height}" radius="${hexagon_side * 1.1547}"/> <!-- sqrt(4/3) * side for circumradius -->
       </geometry>
       <material name="blue">
         <color rgba="0.2 0.3 0.8 1.0"/>
       </material>
-    </visual>
-    <collision>
-      <geometry>
-        <cylinder length="${base_height}" radius="${base_radius}"/>
-      </geometry>
+      <origin xyz="0 0 ${base_height/2}" rpy="0 0 0"/>
+    </visual>
+    <collision>
+      <geometry>
+        <!-- Hexagonal prism approximation using cylinder -->
+        <cylinder length="${base_height}" radius="${hexagon_side * 1.1547}"/>
+      </geometry>
+      <origin xyz="0 0 ${base_height/2}" rpy="0 0 0"/>
     </collision>
     <inertial>
       <mass value="10.0"/>
-      <inertia ixx="0.1" ixy="0.0" ixz="0.0"
-               iyy="0.1" iyz="0.0"
-               izz="0.2"/>
+      <!-- Hexagonal inertia calculation -->
+      <inertia ixx="0.15" ixy="0.0" ixz="0.0"
+               iyy="0.15" iyz="0.0"
+               izz="0.25"/>
+      <origin xyz="0 0 ${base_height/2}" rpy="0 0 0"/>
     </inertial>
   </link>
@@ -117,46 +127,46 @@
     </xacro:if>
   </xacro:macro>
-  <!-- Create three omni wheels -->
-  <xacro:omni_wheel name="wheel_1" x="${wheel_1_x}" y="${wheel_1_y}"/>
-  <xacro:omni_wheel name="wheel_2" x="${wheel_2_x}" y="${wheel_2_y}"/>
-  <xacro:omni_wheel name="wheel_3" x="${wheel_3_x}" y="${wheel_3_y}"/>
-  <!-- LIDAR frame -->
-  <link name="lidar_frame">
-    <visual>
-      <geometry>
-        <cylinder length="0.05" radius="0.08"/>
-      </geometry>
-      <material name="red">
-        <color rgba="0.8 0.2 0.2 1.0"/>
-      </material>
-      <origin xyz="0 0 0" rpy="0 0 0"/>
-    </visual>
-    <collision>
-      <geometry>
-        <cylinder length="0.05" radius="0.08"/>
-      </geometry>
-      <origin xyz="0 0 0" rpy="0 0 0"/>
-    </collision>
-    <inertial>
-      <mass value="0.2"/>
-      <inertia ixx="0.001" ixy="0.0" ixz="0.0"
-               iyy="0.001" iyz="0.0"
-               izz="0.002"/>
-    </inertial>
-  </link>
-  <joint name="lidar_joint" type="fixed">
+  <!-- Create three omni wheels (lf, rf, b) -->
+  <xacro:omni_wheel name="wheel_lf" x="${wheel_lf_x}" y="${wheel_lf_y}"/>
+  <xacro:omni_wheel name="wheel_rf" x="${wheel_rf_x}" y="${wheel_rf_y}"/>
+  <xacro:omni_wheel name="wheel_b" x="${wheel_b_x}" y="${wheel_b_y}"/>
+  <!-- TF-Luna Single-Point LIDAR -->
+  <link name="tf_luna_link">
+    <visual>
+      <geometry>
+        <cylinder length="0.035" radius="0.012"/>
+      </geometry>
+      <material name="dark_red">
+        <color rgba="0.6 0.1 0.1 1.0"/>
+      </material>
+      <origin xyz="0 0 0" rpy="0 0 0"/>
+    </visual>
+    <collision>
+      <geometry>
+        <cylinder length="0.035" radius="0.012"/>
+      </geometry>
+      <origin xyz="0 0 0" rpy="0 0 0"/>
+    </collision>
+    <inertial>
+      <mass value="0.015"/>
+      <inertia ixx="0.000005" ixy="0.0" ixz="0.0"
+               iyy="0.000005" iyz="0.0"
+               izz="0.00001"/>
+    </inertial>
+  </link>
+  <joint name="tf_luna_joint" type="fixed">
     <parent link="base_link"/>
-    <child link="lidar_frame"/>
-    <origin xyz="0 0 ${base_height + 0.05}" rpy="0 0 0"/>
+    <child link="tf_luna_link"/>
+    <origin xyz="0.15 0 ${base_height + 0.02}" rpy="0 0 0"/>
   </joint>
-  <!-- Ultrasonic Sensors (4x) -->
-  <xacro:macro name="ultrasonic_sensor" params="name x y z">
+  <!-- Laser Distance Sensors (6x - 2 per side for wall alignment) -->
+  <xacro:macro name="laser_distance_sensor" params="name x y z">
     <link name="${name}_link">
       <visual>
         <geometry>
-          <cylinder length="0.02" radius="0.015"/>
-        </geometry>
-        <material name="yellow">
-          <color rgba="1.0 1.0 0.0 1.0"/>
+          <cylinder length="0.03" radius="0.012"/>
+        </geometry>
+        <material name="red">
+          <color rgba="0.8 0.1 0.1 1.0"/>
         </material>
         <origin xyz="0 0 0" rpy="0 0 0"/>
@@ -164,13 +174,13 @@
       <collision>
         <geometry>
-          <cylinder length="0.02" radius="0.015"/>
+          <cylinder length="0.03" radius="0.012"/>
         </geometry>
         <origin xyz="0 0 0" rpy="0 0 0"/>
       </collision>
       <inertial>
-        <mass value="0.05"/>
-        <inertia ixx="0.0001" ixy="0.0" ixz="0.0"
-                 iyy="0.0001" iyz="0.0"
-                 izz="0.0002"/>
+        <mass value="0.04"/>
+        <inertia ixx="0.00005" ixy="0.0" ixz="0.0"
+                 iyy="0.00005" iyz="0.0"
+                 izz="0.0001"/>
       </inertial>
     </link>
@@ -181,13 +191,13 @@
     </joint>
   </xacro:macro>
-  <!-- IR Sharp Sensors (3x) -->
-  <xacro:macro name="ir_sensor" params="name x y z">
+  <!-- HC-SR04 Ultrasonic Sensors (2x front) -->
+  <xacro:macro name="hcsr04_sensor" params="name x y z">
     <link name="${name}_link">
       <visual>
         <geometry>
-          <box size="0.02 0.02 0.015"/>
-        </geometry>
-        <material name="orange">
-          <color rgba="1.0 0.5 0.0 1.0"/>
+          <cylinder length="0.025" radius="0.008"/>
+        </geometry>
+        <material name="yellow">
+          <color rgba="1.0 1.0 0.0 1.0"/>
         </material>
         <origin xyz="0 0 0" rpy="0 0 0"/>
@@ -195,5 +205,5 @@
       <collision>
         <geometry>
-          <box size="0.02 0.02 0.015"/>
+          <cylinder length="0.025" radius="0.008"/>
         </geometry>
         <origin xyz="0 0 0" rpy="0 0 0"/>
@@ -201,7 +211,7 @@
       <inertial>
         <mass value="0.03"/>
-        <inertia ixx="0.0001" ixy="0.0" ixz="0.0"
-                 iyy="0.0001" iyz="0.0"
-                 izz="0.0002"/>
+        <inertia ixx="0.00003" ixy="0.0" ixz="0.0"
+                 iyy="0.00003" iyz="0.0"
+                 izz="0.00006"/>
       </inertial>
     </link>
@@ -212,68 +222,80 @@
     </joint>
   </xacro:macro>
-  <!-- Line Sensor -->
-  <link name="line_sensor_link">
-    <visual>
-      <geometry>
-        <box size="0.08 0.03 0.01"/>
-      </geometry>
-      <material name="purple">
-        <color rgba="0.8 0.0 0.8 1.0"/>
-      </material>
-      <origin xyz="0 0 0" rpy="0 0 0"/>
-    </visual>
-    <collision>
-      <geometry>
-        <box size="0.08 0.03 0.01"/>
-      </geometry>
-      <origin xyz="0 0 0" rpy="0 0 0"/>
-    </collision>
-    <inertial>
-      <mass value="0.02"/>
-      <inertia ixx="0.0001" ixy="0.0" ixz="0.0"
-               iyy="0.0001" iyz="0.0"
-               izz="0.0002"/>
-    </inertial>
-  </link>
-  <joint name="line_sensor_joint" type="fixed">
-    <parent link="base_link"/>
-    <child link="line_sensor_link"/>
-    <origin xyz="0 0 -${base_height/2 - 0.02}" rpy="0 0 0"/>
-  </joint>
-  <!-- Create ultrasonic sensors -->
-  <xacro:ultrasonic_sensor name="ultrasonic_front" x="${base_radius - 0.02}" y="0" z="${base_height/2}"/>
-  <xacro:ultrasonic_sensor name="ultrasonic_back" x="${-base_radius + 0.02}" y="0" z="${base_height/2}"/>
-  <xacro:ultrasonic_sensor name="ultrasonic_left" x="0" y="${base_radius - 0.02}" z="${base_height/2}"/>
-  <xacro:ultrasonic_sensor name="ultrasonic_right" x="0" y="${-base_radius + 0.02}" z="${base_height/2}"/>
-  <!-- Create IR sensors -->
-  <xacro:ir_sensor name="ir_front" x="${base_radius - 0.05}" y="0" z="${base_height/2}"/>
-  <xacro:ir_sensor name="ir_left" x="0" y="${base_radius - 0.05}" z="${base_height/2}"/>
-  <xacro:ir_sensor name="ir_right" x="0" y="${-base_radius + 0.05}" z="${base_height/2}"/>
-  <!-- IMU frame -->
-  <link name="imu_link">
-    <visual>
-      <geometry>
-        <box size="0.03 0.03 0.02"/>
+  <!-- Line Sensors (3x individual, assembled side by side) -->
+  <xacro:macro name="line_sensor" params="name x y z">
+    <link name="${name}_link">
+      <visual>
+        <geometry>
+          <box size="0.015 0.08 0.005"/>
+        </geometry>
+        <material name="purple">
+          <color rgba="0.8 0.0 0.8 1.0"/>
+        </material>
+        <origin xyz="0 0 0" rpy="0 0 0"/>
+      </visual>
+      <collision>
+        <geometry>
+          <box size="0.015 0.08 0.005"/>
+        </geometry>
+        <origin xyz="0 0 0" rpy="0 0 0"/>
+      </collision>
+      <inertial>
+        <mass value="0.02"/>
+        <inertia ixx="0.00001" ixy="0.0" ixz="0.0"
+                 iyy="0.00001" iyz="0.0"
+                 izz="0.00002"/>
+      </inertial>
+    </link>
+    <joint name="${name}_joint" type="fixed">
+      <parent link="base_link"/>
+      <child link="${name}_link"/>
+      <origin xyz="${x} ${y} ${z}" rpy="0 0 0"/>
+    </joint>
+  </xacro:macro>
+  <!-- Create laser distance sensors (6x - 2 per side for wall alignment) -->
+  <!-- Left side sensors -->
+  <xacro:laser_distance_sensor name="laser_left_front" x="${hexagon_side * 0.433}" y="${hexagon_side * 0.75}" z="${base_height/2}"/>
+  <xacro:laser_distance_sensor name="laser_left_back" x="${-hexagon_side * 0.433}" y="${hexagon_side * 0.75}" z="${base_height/2}"/>
+  <!-- Right side sensors -->
+  <xacro:laser_distance_sensor name="laser_right_front" x="${hexagon_side * 0.433}" y="${-hexagon_side * 0.75}" z="${base_height/2}"/>
+  <xacro:laser_distance_sensor name="laser_right_back" x="${-hexagon_side * 0.433}" y="${-hexagon_side * 0.75}" z="${base_height/2}"/>
+  <!-- Back side sensors -->
+  <xacro:laser_distance_sensor name="laser_back_left" x="${-hexagon_side}" y="${hexagon_side * 0.25}" z="${base_height/2}"/>
+  <xacro:laser_distance_sensor name="laser_back_right" x="${-hexagon_side}" y="${-hexagon_side * 0.25}" z="${base_height/2}"/>
+  <!-- Create HC-SR04 ultrasonic sensors (2x front) -->
+  <xacro:hcsr04_sensor name="hcsr04_front_left" x="${hexagon_side * 0.866}" y="${hexagon_side * 0.3}" z="${base_height/2}"/>
+  <xacro:hcsr04_sensor name="hcsr04_front_right" x="${hexagon_side * 0.866}" y="${-hexagon_side * 0.3}" z="${base_height/2}"/>
+  <!-- Create line sensors (3x individual, assembled side by side at front) -->
+  <xacro:line_sensor name="line_sensor_left" x="${hexagon_side * 0.95}" y="0.025" z="-${base_height/2 - 0.01}"/>
+  <xacro:line_sensor name="line_sensor_center" x="${hexagon_side * 0.95}" y="0" z="-${base_height/2 - 0.01}"/>
+  <xacro:line_sensor name="line_sensor_right" x="${hexagon_side * 0.95}" y="-0.025" z="-${base_height/2 - 0.01}"/>
+  <!-- MPU6050 IMU -->
+  <link name="mpu6050_link">
+    <visual>
+      <geometry>
+        <box size="0.025 0.015 0.01"/>
       </geometry>
       <material name="green">
         <color rgba="0.2 0.8 0.2 1.0"/>
       </material>
-    </visual>
-    <collision>
-      <geometry>
-        <box size="0.03 0.03 0.02"/>
-      </geometry>
-    </collision>
-    <inertial>
-      <mass value="0.05"/>
-      <inertia ixx="0.0001" ixy="0.0" ixz="0.0"
-               iyy="0.0001" iyz="0.0"
-               izz="0.0002"/>
-    </inertial>
-  </link>
-  <joint name="imu_joint" type="fixed">
+      <origin xyz="0 0 0" rpy="0 0 0"/>
+    </visual>
+    <collision>
+      <geometry>
+        <box size="0.025 0.015 0.01"/>
+      </geometry>
+      <origin xyz="0 0 0" rpy="0 0 0"/>
+    </collision>
+    <inertial>
+      <mass value="0.005"/>
+      <inertia ixx="0.000001" ixy="0.0" ixz="0.0"
+               iyy="0.000001" iyz="0.0"
+               izz="0.000002"/>
+    </inertial>
+  </link>
+  <joint name="mpu6050_joint" type="fixed">
     <parent link="base_link"/>
-    <child link="imu_link"/>
-    <origin xyz="0.05 0 ${base_height - 0.01}" rpy="0 0 0"/>
+    <child link="mpu6050_link"/>
+    <origin xyz="0.05 0 ${base_height - 0.005}" rpy="0 0 0"/>
   </joint>
   <!-- Camera frame -->
@@ -304,9 +326,9 @@
     <origin xyz="${base_radius - 0.02} 0 ${base_height + 0.03}" rpy="0 0 0"/>
   </joint>
-  <!-- Lifter/Forklift (1x DC Motor + Encoder) -->
-  <link name="lifter_link">
-    <visual>
-      <geometry>
-        <box size="0.1 0.1 0.3"/>
+  <!-- Gripper Assembly Base (DC Motor for up/down movement) -->
+  <link name="gripper_base_link">
+    <visual>
+      <geometry>
+        <box size="0.12 0.08 0.15"/>
       </geometry>
       <material name="silver">
@@ -317,31 +339,153 @@
     <collision>
       <geometry>
-        <box size="0.1 0.1 0.3"/>
-      </geometry>
-      <origin xyz="0 0 0" rpy="0 0 0"/>
-    </collision>
-    <inertial>
-      <mass value="2.0"/>
-      <inertia ixx="0.1" ixy="0.0" ixz="0.0"
-               iyy="0.1" iyz="0.0"
-               izz="0.05"/>
-    </inertial>
-  </link>
-  <joint name="lifter_joint" type="prismatic">
+        <box size="0.12 0.08 0.15"/>
+      </geometry>
+      <origin xyz="0 0 0" rpy="0 0 0"/>
+    </collision>
+    <inertial>
+      <mass value="1.5"/>
+      <inertia ixx="0.05" ixy="0.0" ixz="0.0"
+               iyy="0.05" iyz="0.0"
+               izz="0.03"/>
+    </inertial>
+  </link>
+  <joint name="gripper_base_joint" type="prismatic">
     <parent link="base_link"/>
-    <child link="lifter_link"/>
-    <origin xyz="0 0 ${base_height/2}" rpy="0 0 0"/>
+    <child link="gripper_base_link"/>
+    <origin xyz="0.15 0 ${base_height/2}" rpy="0 0 0"/>
     <axis xyz="0 0 1"/>
-    <limit effort="100.0" lower="0.0" upper="0.1" velocity="0.1"/>
+    <limit effort="50.0" lower="0.0" upper="0.2" velocity="0.15"/>
   </joint>
-  <!-- Servo Motors (5x) -->
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