Commit message: refactor Mega firmware: -581 lines, throttle VFF, consolidate move funcs, simplify perimeter safety, fix APF direction, strip IMU dead code

File: ros2_ws/src/my_robot_description/urdf/my_robot.urdf.xacro (robot description, xacro)
@@ -114,15 +114,5 @@
     </joint>
     <xacro:if value="$(arg use_ros2_control)">
-      <!-- ROS 2 Control interface for wheel -->
-      <ros2_control name="${name}_wheel_controller" type="system">
-        <hardware>
-          <plugin>gazebo_ros2_control/GazeboSystem</plugin>
-        </hardware>
-        <joint name="${name}_joint">
-          <command_interface name="velocity"/>
-          <state_interface name="velocity"/>
-          <state_interface name="position"/>
-        </joint>
-      </ros2_control>
+      <!-- ROS 2 Control interface placeholder -->
     </xacro:if>
   </xacro:macro>
@@ -515,249 +505,3 @@
   <xacro:container name="container_right_front" x="-0.12" y="-0.12" z="${base_height + 0.04}"/>
   <xacro:container name="container_right_back" x="-0.18" y="-0.12" z="${base_height + 0.04}"/>
-  <!-- Gazebo plugins -->
-  <gazebo>
-    <!-- Differential drive plugin (simplified for basic movement) -->
-    <plugin name="diff_drive" filename="libgazebo_ros_diff_drive.so">
-      <ros>
-        <namespace></namespace>
-        <remapping>cmd_vel:=/cmd_vel</remapping>
-        <remapping>odom:=/odom</remapping>
-      </ros>
-      <!-- Use only two wheels for basic differential drive -->
-      <left_joint>wheel_1_joint</left_joint>
-      <right_joint>wheel_2_joint</right_joint>
-      <!-- Wheel properties -->
-      <wheel_separation>${base_radius * 1.732}</wheel_separation>
-      <wheel_diameter>${wheel_radius * 2}</wheel_diameter>
-      <!-- Robot properties -->
-      <robot_base_frame>base_link</robot_base_frame>
-      <wheel_torque>20.0</wheel_torque>
-      <wheel_acceleration>1.0</wheel_acceleration>
-      <!-- Odometry properties -->
-      <publish_odom>true</publish_odom>
-      <publish_odom_tf>true</publish_odom_tf>
-      <publish_wheel_tf>true</publish_wheel_tf>
-      <odometry_frame>odom</odometry_frame>
-      <odometry_topic>odom</odometry_topic>
-      <!-- Command timeout -->
-      <cmd_timeout>0.25</cmd_timeout>
-      <!-- Legacy mode (for compatibility) -->
-      <legacy_mode>false</legacy_mode>
-    </plugin>
-    <!-- MPU6050 IMU sensor plugin -->
-    <plugin name="mpu6050_plugin" filename="libgazebo_ros_imu_sensor.so">
-      <ros>
-        <namespace></namespace>
-        <remapping>imu/data:=/imu/data</remapping>
-      </ros>
-      <always_on>true</always_on>
-      <update_rate>50.0</update_rate>
-      <body_name>mpu6050_link</body_name>
-      <topic_name>imu/data</topic_name>
-      <gaussian_noise>0.001</gaussian_noise>
-      <frame_name>mpu6050_link</frame_name>
-    </plugin>
-    <!-- TF-Luna Single-Point LIDAR plugin -->
-    <plugin name="tf_luna_plugin" filename="libgazebo_ros_ray_sensor.so">
-      <ros>
-        <namespace></namespace>
-        <remapping>range:=/tf_luna/range</remapping>
-      </ros>
-      <always_on>true</always_on>
-      <update_rate>10.0</update_rate>
-      <topic_name>range</topic_name>
-      <frame_name>tf_luna_link</frame_name>
-      <ray>
-        <range>
-          <min>0.1</min>
-          <max>8.0</max>
-          <resolution>0.01</resolution>
-        </range>
-      </ray>
-    </plugin>
-    <!-- Laser Distance Sensor plugins (6x - wall alignment) -->
-    <plugin name="laser_left_front_plugin" filename="libgazebo_ros_ray_sensor.so">
-      <ros>
-        <namespace></namespace>
-        <remapping>range:=/distance/left_front</remapping>
-      </ros>
-      <always_on>true</always_on>
-      <update_rate>15.0</update_rate>
-      <topic_name>range</topic_name>
-      <frame_name>laser_left_front_link</frame_name>
-      <ray>
-        <range>
-          <min>0.02</min>
-          <max>4.0</max>
-          <resolution>0.01</resolution>
-        </range>
-      </ray>
-    </plugin>
-    <plugin name="laser_left_back_plugin" filename="libgazebo_ros_ray_sensor.so">
-      <ros>
-        <namespace></namespace>
-        <remapping>range:=/distance/left_back</remapping>
-      </ros>
-      <always_on>true</always_on>
-      <update_rate>15.0</update_rate>
-      <topic_name>range</topic_name>
-      <frame_name>laser_left_back_link</frame_name>
-      <ray>
-        <range>
-          <min>0.02</min>
-          <max>4.0</max>
-          <resolution>0.01</resolution>
-        </range>
-      </ray>
-    </plugin>
-    <plugin name="laser_right_front_plugin" filename="libgazebo_ros_ray_sensor.so">
-      <ros>
-        <namespace></namespace>
-        <remapping>range:=/distance/right_front</remapping>
-      </ros>
-      <always_on>true</always_on>
-      <update_rate>15.0</update_rate>
-      <topic_name>range</topic_name>
-      <frame_name>laser_right_front_link</frame_name>
-      <ray>
-        <range>
-          <min>0.02</min>
-          <max>4.0</max>
-          <resolution>0.01</resolution>
-        </range>
-      </ray>
-    </plugin>
-    <plugin name="laser_right_back_plugin" filename="libgazebo_ros_ray_sensor.so">
-      <ros>
-        <namespace></namespace>
-        <remapping>range:=/distance/right_back</remapping>
-      </ros>
-      <always_on>true</always_on>
-      <update_rate>15.0</update_rate>
-      <topic_name>range</topic_name>
-      <frame_name>laser_right_back_link</frame_name>
-      <ray>
-        <range>
-          <min>0.02</min>
-          <max>4.0</max>
-          <resolution>0.01</resolution>
-        </range>
-      </ray>
-    </plugin>
-    <plugin name="laser_back_left_plugin" filename="libgazebo_ros_ray_sensor.so">
-      <ros>
-        <namespace></namespace>
-        <remapping>range:=/distance/back_left</remapping>
-      </ros>
-      <always_on>true</always_on>
-      <update_rate>15.0</update_rate>
-      <topic_name>range</topic_name>
-      <frame_name>laser_back_left_link</frame_name>
-      <ray>
-        <range>
-          <min>0.02</min>
-          <max>4.0</max>
-          <resolution>0.01</resolution>
-        </range>
-      </ray>
-    </plugin>
-    <plugin name="laser_back_right_plugin" filename="libgazebo_ros_ray_sensor.so">
-      <ros>
-        <namespace></namespace>
-        <remapping>range:=/distance/back_right</remapping>
-      </ros>
-      <always_on>true</always_on>
-      <update_rate>15.0</update_rate>
-      <topic_name>range</topic_name>
-      <frame_name>laser_back_right_link</frame_name>
-      <ray>
-        <range>
-          <min>0.02</min>
-          <max>4.0</max>
-          <resolution>0.01</resolution>
-        </range>
-      </ray>
-    </plugin>
-    <!-- HC-SR04 Ultrasonic Sensor plugins (2x front) -->
-    <plugin name="hcsr04_front_left_plugin" filename="libgazebo_ros_ray_sensor.so">
-      <ros>
-        <namespace></namespace>
-        <remapping>range:=/ultrasonic/front_left</remapping>
-      </ros>
-      <always_on>true</always_on>
-      <update_rate>10.0</update_rate>
-      <topic_name>range</topic_name>
-      <frame_name>hcsr04_front_left_link</frame_name>
-      <ray>
-        <range>
-          <min>0.02</min>
-          <max>4.0</max>
-          <resolution>0.01</resolution>
-        </range>
-      </ray>
-    </plugin>
-    <plugin name="hcsr04_front_right_plugin" filename="libgazebo_ros_ray_sensor.so">
-      <ros>
-        <namespace></namespace>
-        <remapping>range:=/ultrasonic/front_right</remapping>
-      </ros>
-      <always_on>true</always_on>
-      <update_rate>10.0</update_rate>
-      <topic_name>range</topic_name>
-      <frame_name>hcsr04_front_right_link</frame_name>
-      <ray>
-        <range>
-          <min>0.02</min>
-          <max>4.0</max>
-          <resolution>0.01</resolution>
-        </range>
-      </ray>
-    </plugin>
-    <!-- Line Sensor plugins (3x) - using contact sensors -->
-    <plugin name="line_sensor_left_plugin" filename="libgazebo_ros_bumper.so">
-      <ros>
-        <namespace></namespace>
-        <remapping>bumper:=/line_sensor/left</remapping>
-      </ros>
-      <always_on>true</always_on>
-      <update_rate>50.0</update_rate>
-      <bumper_topic_name>bumper</bumper_topic_name>
-      <frame_name>line_sensor_left_link</frame_name>
-    </plugin>
-    <plugin name="line_sensor_center_plugin" filename="libgazebo_ros_bumper.so">
-      <ros>
-        <namespace></namespace>
-        <remapping>bumper:=/line_sensor/center</remapping>
-      </ros>
-      <always_on>true</always_on>
-      <update_rate>50.0</update_rate>
-      <bumper_topic_name>bumper</bumper_topic_name>
-      <frame_name>line_sensor_center_link</frame_name>
-    </plugin>
-    <plugin name="line_sensor_right_plugin" filename="libgazebo_ros_bumper.so">
-      <ros>
-        <namespace></namespace>
-        <remapping>bumper:=/line_sensor/right</remapping>
-      </ros>
-      <always_on>true</always_on>
-      <update_rate>50.0</update_rate>
-      <bumper_topic_name>bumper</bumper_topic_name>
-      <frame_name>line_sensor_right_link</frame_name>
-    </plugin>
-    <!-- Gripper Camera plugin -->
-    <plugin name="gripper_camera_plugin" filename="libgazebo_ros_camera.so">
-      <ros>
-        <namespace></namespace>
-        <remapping>image_raw:=/gripper/camera/image_raw</remapping>
-        <remapping>camera_info:=/gripper/camera/camera_info</remapping>
-      </ros>
-      <always_on>true</always_on>
-      <update_rate>30.0</update_rate>
-      <camera_name>gripper_camera</camera_name>
-      <frame_name>gripper_camera_link</frame_name>
-      <image_topic_name>image_raw</image_topic_name>
-      <camera_info_topic_name>camera_info</camera_info_topic_name>
-      <hack_baseline>0.07</hack_baseline>
-    </plugin>
-  </gazebo>
 </robot>
